File: rp2350_driver.kicad_pcb (KiCad board)
At the start: 6 copper layers, 76 x 46.4 mm, 291 parts, among them J1 XT30, J10 Power Output, J11 CAN2 PLUG, J12 Conn_01x06, J2 XT30, J3 USB_C_Receptacle_USB2.0, J4 SM03B-SRSS-TB, J5 Estop Conn, J6 SM03B-SRSS-TB, J7 Conn_01x03, J8 Conn_01x03, J9 XT30, Q1 Q_PNP_BEC, Q2 Q_PNP_BEC, Q3 Q_PNP_BEC, Q4 Q_PNP_BEC, Q5 Q_NMOS_GDS, SW1 Button, SW2 Button, U1 EG3113, U10 INA240A1D, U101 FUSB302BMPX, U11 USBLC6-2P6, U12 EG3113, U13 TS5A3159DCK, U14 TS5A3159DCK, U15 TS5A3159DCK, U16 CA-IS3052CG, U17 TS5A3159DCK, U18 SIT3088ETK, U19 SIT3088ETK, U2 TX4137, U20 SIT3088ETK, U21 SIT3088ETK, U22 TS5A3159DCK, U23 TS5A3159DCK, U24 TS5A3159DCK, U25 TS5A3159DCK, U26 TS5A3159DCK, U27 TS5A3159DCK, U29 LM74700, U3 W25Q16JV, U4 SPX3819M5-L-3-3, U5 INA240A1D, U6 EG3113, U7 EG3113, U8 RP2350_80QFN, U9 INA240A1D, Y1 ABM8-272-T3

Commit message: Silly but complete routing of the 80v power supply
Parts:
- removed D2: 3.3v Zener, Diode_SMD:D_SOD-123
- removed D8: SS310, Diode_SMD:D_SOD-123F
- removed L1: 22uH 680mA, parts:IND-SMD_L3.0-W3.0_FNR30XXS
- removed R16: 23.7k, Resistor_SMD:R_0402_1005Metric
- removed R19: 124k, Resistor_SMD:R_0402_1005Metric
- removed R3, R4: 50k 0.1%, Resistor_SMD:R_0603_1608Metric
- removed U2: TX4137, Package_TO_SOT_SMD:SOT-23-6
- added C80: 220uF 63V solid, Capacitor_THT:CP_Radial_D10.0mm_P5.00mm, F.Cu at (154.0, 99.6)
- added C81: 1uf 100v, Capacitor_SMD:C_0603_1608Metric, B.Cu at (165.0, 109.0)
- added D4: SS210, Diode_SMD:D_SMA, B.Cu at (159.1, 100.9)
- added JP1: Jumper_2_Open, Jumper:SolderJumper-2_P1.3mm_Bridged_RoundedPad1.0x1.5mm, B.Cu at (164.2, 111.9)
- added L3: 47uH 1A, Inductor_SMD:L_APV_ANR5045, B.Cu at (156.8, 109.4)
- added R5: 10k, Resistor_SMD:R_0402_1005Metric, B.Cu at (152.0, 110.1)
- added R6: 3.3k, Resistor_SMD:R_0402_1005Metric, B.Cu at (150.2, 109.6)
- added U28: XL7005A, Package_SO:SOIC-8-1EP_3.9x4.9mm_P1.27mm_EP2.29x3mm, B.Cu at (162.5, 103.8)
- C11: value 10u 25v -> 100uF ±20% 10V; footprint Capacitor_SMD:C_0805_2012Metric -> Capacitor_SMD:CP_Elec_5x5.4
- C3: value 4.7uF 100v -> 33n; footprint Capacitor_SMD:C_1210_3225Metric -> Capacitor_SMD:C_0402_1005Metric
- C39: value 220uF 63V solid -> 100uF 100V
- C52, U15: moved to F.Cu
- D10, D14, D18, D3: value FR107 -> DSS110; footprint Diode_SMD:D_SOD-123 -> Diode_SMD:D_SOD-123F
- D5: value SMDJ51CA -> SMDJ85A
- R25, R41, R73, R9: value 0R -> 4.7R
- moved C11 13.7 mm to (151.2, 104.4), turned to 90 degrees
- moved C42 8.00 mm to (161.7, 109.7), turned to 45 degrees
- moved C47 7.59 mm to (162.7, 101.5), turned to 180 degrees
- moved R8 5.05 mm to (166.3, 113.6)
- moved C52 4.45 mm to (163.5, 98.3), turned to -90 degrees
- moved C3 4.36 mm to (152.0, 109.1), turned to 180 degrees
- moved U15 4.21 mm to (161.2, 98.8), turned to 0 degrees
- moved TP8 3.46 mm to (161.7, 115.8), turned to -90 degrees
- moved TP12 2.19 mm to (165.0, 98.9)
- moved C4 1.27 mm to (169.7, 110.2)
- moved TP14 0.71 mm to (172.5, 107.8)
- moved C39 0.58 mm to (151.9, 112.7), turned to -15 degrees
- moved TP15 0.46 mm to (173.4, 105.8)
- moved U3 0.32 mm to (171.0, 108.9)
- moved R25 0.20 mm to (148.0, 99.8)
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Connections:
- C3 pad 1: VMOT -> Vdrive
- C3 pad 2: GND -> Net-(U28-FB)
- C78 pad 2: VMOT -> Net-(JP1-A)
- Q5 pad 2: VMOT -> Net-(JP1-A)
- U29 pad 4: VMOT -> Net-(JP1-A)
Routing:
- net Net-(JP1-A): track 0.00 -> 23.8 mm
- net /V_ENABLE: track 23.2 -> 0.00 mm, vias 2 -> 0
- net VMOT: track 56.1 -> 36.5 mm
- net GND: track 205.1 -> 223.1 mm, vias 245 -> 238
- net Net-(U28-FB): track 0.00 -> 13.7 mm, vias 0 -> 2
- net Vdrive: track 236.3 -> 245.4 mm
- net /TH_SW_1: track 27.8 -> 22.2 mm, vias 3 -> 2
- net +3V3: track 260.9 -> 255.5 mm, vias 18 -> 17
- net /MOT_TH: track 58.8 -> 64.1 mm, vias 2 -> 1
- net /ENC_C_DATA: track 84.4 -> 80.6 mm
- net /TH1_SENSE: track 22.3 -> 18.9 mm, vias 2 -> 1
- net Net-(U2-FB): track 2.98 -> 0.00 mm
- net A_PWM_H: track 45.0 -> 47.9 mm, vias 3 -> 2
- net /QSPI_SD1: track 8.38 -> 10.2 mm
- net Net-(R3-Pad2): track 1.77 -> 0.00 mm
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- added copper zone on B.Cu, net Net-(D4-K)
- removed copper zone on B.Cu, net Net-(D8-K)
- removed copper zone on B.Cu, net VMOT

Commit message: minor tweaks
Parts:
- moved C59 1.74 mm to (158.2, 125.4)
- moved U17 1.63 mm to (156.1, 125.7)
Routing:
- net Vdrive: track 245.4 -> 242.9 mm
- net /V_SW: track 42.4 -> 44.2 mm
- net /V_ENC: track 35.1 -> 34.0 mm
- net +3V3: track 255.5 -> 256.6 mm
- net /I2C_SDA: track 116.1 -> 117.0 mm
- net /ENC_D_DATA: track 82.9 -> 83.5 mm
- net /ENC_B_SW: track 110.3 -> 110.8 mm

Commit message: Whether inadvisedly or not, I have ordered this rev
Routing:
- net Vdrive: track 242.9 -> 246.6 mm
- net /H1_SW: track 87.0 -> 87.6 mm
Other:
- board text added: "80V max"
