File: hardware/rp2350_driver.kicad_pcb (KiCad board)
At the start: 6 copper layers, 76 x 46.4 mm, 291 parts, among them J1 XT30, J10 Power Output, J11 CAN2 PLUG, J12 Conn_01x06, J2 XT30, J3 USB_C_Receptacle_USB2.0, J4 SM03B-SRSS-TB, J5 Estop Conn, J6 SM03B-SRSS-TB, J7 Conn_01x03, J8 Conn_01x03, J9 XT30, Q1 Q_PNP_BEC, Q2 Q_PNP_BEC, Q3 Q_PNP_BEC, Q4 Q_PNP_BEC, Q5 Q_NMOS_GDS, SW1 Button, SW2 Button, U1 EG3113, U10 INA240A1D, U101 FUSB302BMPX, U11 USBLC6-2P6, U12 EG3113, U13 TS5A3159DCK, U14 TS5A3159DCK, U15 TS5A3159DCK, U16 CA-IS3052CG, U17 TS5A3159DCK, U18 SIT3088ETK, U19 SIT3088ETK, U20 SIT3088ETK, U21 SIT3088ETK, U22 TS5A3159DCK, U23 TS5A3159DCK, U24 TS5A3159DCK, U25 TS5A3159DCK, U26 TS5A3159DCK, U27 TS5A3159DCK, U28 XL7005A, U29 LM74700, U3 W25Q16JV, U4 SPX3819M5-L-3-3, U5 INA240A1D, U6 EG3113, U7 EG3113, U8 RP2350_80QFN, U9 INA240A1D, Y1 ABM8-272-T3

Commit message: Fix protection voltage ratings for real 60V operation
- FETs: BSC030N08NS5 (80V, C501507) -> TMG08N10SI (100V, C7422896); same
  PowerPAK SO-8 footprint, already vetted in the JLC cart
- Phase TVS D9/D13/D17/D21: SMAJ51A -> SMAJ64A. 51V standoff sat in
  leakage/breakdown whenever the bus exceeded ~51V with a high side on;
  64V standoff clears a 60V bus
- Bus TVS D5: SMDJ85A -> SMDJ60A. 85V standoff could never clamp before
  the old 80V FETs; 60V standoff clamps ~97V, inside the new FETs' 100V

LCSC numbers for the two new TVS values are marked LCSC-TBD — pick in-stock
parts at order time. Netlist-verified: value-only change, topology untouched.

Co-Authored-By: Claude Fable 5 <noreply@anthropic.com>
Parts:
- AH1, AL1, BH1, BL1, CH1, CH2, CL1, CL2: value MOSFETSO-8 -> TMG08N10SI
- D13, D17, D21, D9: value SMAJ51A -> SMAJ64A
- D5: value SMDJ85A -> SMDJ60A
Changed lines of the file:
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@@
 			)
 		)
-		(property "Value" "SMAJ51A"
+		(property "Value" "SMAJ64A"
 			(at 0 2.600001 0)
 			(layer "F.Fab")
@@
 			)
 		)
-		(property "LCSC" "C366557"
+		(property "LCSC" "LCSC-TBD-SMAJ64A"
 			(at 0 0 0)
 			(layer "F.Fab")
@@
 			)
 		)
-		(property "Value" "MOSFETSO-8"
+		(property "Value" "TMG08N10SI"
 			(at 0 3.5 90)
 			(layer "F.Fab")
@@
 			)
 		)
-		(property "LCSC" "C501507"
+		(property "LCSC" "C7422896"
 			(at 0 0 0)
 			(layer "F.Fab")
@@
 			)
 		)
-		(property "Value" "MOSFETSO-8"
+		(property "Value" "TMG08N10SI"
 			(at 0 3.5 90)
 			(layer "F.Fab")
@@
 			)
 		)
-		(property "LCSC" "C501507"
+		(property "LCSC" "C7422896"
 			(at 0 0 0)
 			(layer "F.Fab")
@@
 			)
 		)
-		(property "Value" "MOSFETSO-8"
+		(property "Value" "TMG08N10SI"
 			(at 0 3.5 0)
 			(layer "F.Fab")
@@
 			)
 		)
-		(property "LCSC" "C501507"
+		(property "LCSC" "C7422896"
 			(at 0 0 0)
 			(layer "F.Fab")
@@
 			)
 		)
-		(property "Value" "MOSFETSO-8"
+		(property "Value" "TMG08N10SI"
 			(at 0 3.5 0)
 			(layer "F.Fab")
@@
 			)
 		)
-		(property "LCSC" "C501507"
+		(property "LCSC" "C7422896"
 			(at 0 0 0)
 			(layer "F.Fab")
@@
 			)
 		)
-		(property "Value" "MOSFETSO-8"
+		(property "Value" "TMG08N10SI"
 			(at 0 3.5 90)
 			(layer "F.Fab")
@@
 			)
 		)
-		(property "LCSC" "C501507"
+		(property "LCSC" "C7422896"
 			(at 0 0 0)
 			(layer "F.Fab")
@@
 			)
 		)
-		(property "Value" "MOSFETSO-8"
+		(property "Value" "TMG08N10SI"
 			(at 0 3.5 0)
 			(layer "F.Fab")
@@
 			)
 		)
-		(property "LCSC" "C501507"
+		(property "LCSC" "C7422896"
 			(at 0 0 0)
 			(layer "F.Fab")
@@
 			)
 		)
-		(property "Value" "SMAJ51A"
+		(property "Value" "SMAJ64A"
 			(at 0 2.600001 0)
 			(layer "F.Fab")
@@
 			)
 		)
-		(property "LCSC" "C366557"
+		(property "LCSC" "LCSC-TBD-SMAJ64A"
 			(at 0 0 180)
 			(unlocked yes)
@@
 			)
 		)
-		(property "Value" "MOSFETSO-8"
+		(property "Value" "TMG08N10SI"
 			(at 0 3.5 90)
 			(layer "F.Fab")
@@
 			)
 		)
-		(property "LCSC" "C501507"
+		(property "LCSC" "C7422896"
 			(at 0 0 90)
 			(layer "F.Fab")
@@
 			)
 		)
-		(property "Value" "SMAJ51A"
+		(property "Value" "SMAJ64A"
 			(at 0 2.6 0)
 			(layer "F.Fab")
@@
 			)
 		)
-		(property "LCSC" "C366557"
+		(property "LCSC" "LCSC-TBD-SMAJ64A"
 			(at 0 0 0)
 			(layer "F.Fab")
@@
 			)
 		)
-		(property "Value" "MOSFETSO-8"
+		(property "Value" "TMG08N10SI"
 			(at 0 3.5 180)
 			(layer "F.Fab")
@@
 			)
 		)
-		(property "LCSC" "C501507"
+		(property "LCSC" "C7422896"
 			(at 0 0 0)
 			(layer "F.Fab")
@@
 			)
 		)
-		(property "Value" "SMAJ51A"
+		(property "Value" "SMAJ64A"
 			(at 0 2.600001 0)
 			(layer "F.Fab")
@@
 			)
 		)
-		(property "LCSC" "C366557"
+		(property "LCSC" "LCSC-TBD-SMAJ64A"
 			(at 0 0 0)
 			(layer "F.Fab")
@@
 			)
 		)
-		(property "Value" "SMDJ85A"
+		(property "Value" "SMDJ60A"
 			(at 0 -4.199999 0)
 			(layer "B.Fab")
@@
 			)
 		)
-		(property "LCSC" "C2990214"
+		(property "LCSC" "LCSC-TBD-SMDJ60A"
 			(at 0 0 0)
 			(layer "B.Fab")

Commit message: Correct bridge FET part; map R82-R85 pins to preserve existing copper
- Bridge FETs: TMG08N10SI was wrong -- C7422896 is the SOT-89 FET already
  used at Q5 (LM74700 ideal diode), not a PowerPAK part. Bridge is now
  BSC040N10NS5 (Infineon OptiMOS 100V, PowerPAK SO-8), LCSC marked TBD for
  verification at order time
- R82-R85 pin1 now stays on the transceiver B line (its existing PCB stub
  is untouched); only pin2 moves to the new TERM_x_R switch net, so the
  board edit is a single cut per channel

Co-Authored-By: Claude Fable 5 <noreply@anthropic.com>
Parts:
- AH1, AL1, BH1, BL1, CH1, CH2, CL1, CL2: value TMG08N10SI -> BSC040N10NS5
Changed lines of the file:
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@@
 			)
 		)
-		(property "Value" "TMG08N10SI"
+		(property "Value" "BSC040N10NS5"
 			(at 0 3.5 90)
 			(layer "F.Fab")
@@
 			)
 		)
-		(property "LCSC" "C7422896"
+		(property "LCSC" "LCSC-TBD-BSC040N10NS5"
 			(at 0 0 0)
 			(layer "F.Fab")
@@
 			)
 		)
-		(property "Value" "TMG08N10SI"
+		(property "Value" "BSC040N10NS5"
 			(at 0 3.5 90)
 			(layer "F.Fab")
@@
 			)
 		)
-		(property "LCSC" "C7422896"
+		(property "LCSC" "LCSC-TBD-BSC040N10NS5"
 			(at 0 0 0)
 			(layer "F.Fab")
@@
 			)
 		)
-		(property "Value" "TMG08N10SI"
+		(property "Value" "BSC040N10NS5"
 			(at 0 3.5 0)
 			(layer "F.Fab")
@@
 			)
 		)
-		(property "LCSC" "C7422896"
+		(property "LCSC" "LCSC-TBD-BSC040N10NS5"
 			(at 0 0 0)
 			(layer "F.Fab")
@@
 			)
 		)
-		(property "Value" "TMG08N10SI"
+		(property "Value" "BSC040N10NS5"
 			(at 0 3.5 0)
 			(layer "F.Fab")
@@
 			)
 		)
-		(property "LCSC" "C7422896"
+		(property "LCSC" "LCSC-TBD-BSC040N10NS5"
 			(at 0 0 0)
 			(layer "F.Fab")
@@
 			)
 		)
-		(property "Value" "TMG08N10SI"
+		(property "Value" "BSC040N10NS5"
 			(at 0 3.5 90)
 			(layer "F.Fab")
@@
 			)
 		)
-		(property "LCSC" "C7422896"
+		(property "LCSC" "LCSC-TBD-BSC040N10NS5"
 			(at 0 0 0)
 			(layer "F.Fab")
@@
 			)
 		)
-		(property "Value" "TMG08N10SI"
+		(property "Value" "BSC040N10NS5"
 			(at 0 3.5 0)
 			(layer "F.Fab")
@@
 			)
 		)
-		(property "LCSC" "C7422896"
+		(property "LCSC" "LCSC-TBD-BSC040N10NS5"
 			(at 0 0 0)
 			(layer "F.Fab")
@@
 			)
 		)
-		(property "Value" "TMG08N10SI"
+		(property "Value" "BSC040N10NS5"
 			(at 0 3.5 90)
 			(layer "F.Fab")
@@
 			)
 		)
-		(property "LCSC" "C7422896"
+		(property "LCSC" "LCSC-TBD-BSC040N10NS5"
 			(at 0 0 90)
 			(layer "F.Fab")
@@
 			)
 		)
-		(property "Value" "TMG08N10SI"
+		(property "Value" "BSC040N10NS5"
 			(at 0 3.5 180)
 			(layer "F.Fab")
@@
 			)
 		)
-		(property "LCSC" "C7422896"
+		(property "LCSC" "LCSC-TBD-BSC040N10NS5"
 			(at 0 0 0)
 			(layer "F.Fab")

Commit message: Board: rev-B nets, new parts placed, encoder-corner cluster relaxed
Applies the rev-B schematic to the layout — this is a mid-rework state
that needs an interactive re-route session in the encoder corner:

- Nets renamed (ENC_x_TRX_A/B, TERM_SW) and created (TERM_x_R, LED_VDD);
  R82-R85 pad 2 and D1 VDD cut from their old nets with the through-paths
  bridged
- 28 new footprints placed and netted: U30-U33 termination switches,
  R97-R100 pull-ups, C110-C114, R101-R112 pull-downs, D30, R113, Q6
- 49 encoder-corner parts moved per the courtyard relaxation
  (review/tools/jiggle_result.json); corner signal routing (~570 segments
  + local vias) removed for re-route; stale copper and 12 orphaned vias
  cleaned; zones refilled

Known state (DRC): 214 unconnected airwires = the re-route worklist;
22 shorting + 11 courtyard items, all sub-mm placement seams in the
relaxed corner (drag-to-fix during re-route); 5 proximity items against
protected phase/VMOT copper left untouched deliberately; silk/mask items
cosmetic. U31 parked at (149.5,119.75) pending a better home near R83.

Co-Authored-By: Claude Fable 5 <noreply@anthropic.com>
Parts:
- added C110: 100n, C_0402_1005Metric, B.Cu at (117.2, 110.5)
- added C111: 100n, C_0402_1005Metric, B.Cu at (127.2, 126.4)
- added C112: 100n, C_0402_1005Metric, B.Cu at (127.5, 107.6)
- added C113: 100n, C_0402_1005Metric, B.Cu at (117.0, 103.8)
- added C114: 100n, C_0402_1005Metric, B.Cu at (180.0, 87.5)
- added D30: DSS110, D_SOD-123F, B.Cu at (184.0, 85.5)
- added Q6: Q_NMOS_GDS, SOT-89-3, F.Cu at (184.5, 84.0)
- added R100: 10k, R_0402_1005Metric, B.Cu at (114.5, 102.3)
- added R101: 100k, R_0402_1005Metric, B.Cu at (134.5, 118.0)
- added R102: 100k, R_0402_1005Metric, B.Cu at (131.5, 118.0)
- added R103: 100k, R_0402_1005Metric, B.Cu at (141.0, 107.0)
- added R104: 100k, R_0402_1005Metric, B.Cu at (130.5, 105.5)
- added R105: 100k, R_0402_1005Metric, B.Cu at (133.5, 126.5)
- added R106: 100k, R_0402_1005Metric, B.Cu at (130.5, 126.5)
- added R107: 100k, R_0402_1005Metric, B.Cu at (129.0, 95.0)
- added R108: 100k, R_0402_1005Metric, B.Cu at (161.5, 115.0)
- added R109: 100k, R_0402_1005Metric, B.Cu at (131.5, 84.0)
- added R110: 100k, R_0402_1005Metric, B.Cu at (174.0, 126.0)
- added R111: 100k, R_0402_1005Metric, B.Cu at (177.0, 126.0)
- added R112: 100k, R_0402_1005Metric, B.Cu at (176.5, 84.0)
- added R113: 10k, R_0402_1005Metric, B.Cu at (180.0, 85.0)
- added R97: 10k, R_0402_1005Metric, B.Cu at (118.6, 109.4)
- added R98: 10k, R_0402_1005Metric, B.Cu at (117.1, 126.4)
- added R99: 10k, R_0402_1005Metric, B.Cu at (127.8, 105.6)
- added U30: TS5A3159DCK, SOT-363_SC-70-6, B.Cu at (114.5, 110.5)
- added U31: TS5A3159DCK, SOT-363_SC-70-6, B.Cu at (149.5, 119.8)
- added U32: TS5A3159DCK, SOT-363_SC-70-6, B.Cu at (123.8, 97.8)
- added U33: TS5A3159DCK, SOT-363_SC-70-6, B.Cu at (114.5, 103.8)
- moved R87 2.64 mm to (125.4, 126.4)
- moved R91 2.02 mm to (114.5, 100.0)
- moved C63 2.01 mm to (115.6, 100.0)
- moved R90 1.78 mm to (114.5, 101.5)
- moved R86 1.43 mm to (123.5, 126.4)
- moved R88 1.20 mm to (120.2, 111.9)
- moved R83 1.17 mm to (116.9, 125.1)
- moved U18 1.13 mm to (116.2, 107.6)
- moved R89 0.99 mm to (119.9, 109.9)
- moved R82 0.97 mm to (118.4, 107.8)
- moved D24 0.96 mm to (120.6, 121.7)
- moved U19 0.94 mm to (114.6, 126.4)
- moved D26 0.92 mm to (114.5, 105.5)
- moved R95 0.90 mm to (115.7, 123.4)
- moved FL4 0.90 mm to (117.0, 105.0)
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Connections:
- net Net-(U18-B) renamed /ENC_A_TRX_B
- net Net-(U19-B) renamed /ENC_B_TRX_B
- net Net-(U20-B) renamed /ENC_C_TRX_B
- net Net-(U21-B) renamed /ENC_D_TRX_B
- net Net-(U8-GPIO38) renamed /TERM_SW
- D1 pad 3: Vdrive -> /LED_VDD
- FL1 pad 4: Net-(U19-A) -> /ENC_B_TRX_A
- FL2 pad 4: Net-(U18-A) -> /ENC_A_TRX_A
- FL3 pad 4: Net-(U20-A) -> /ENC_C_TRX_A
- FL4 pad 4: Net-(U21-A) -> /ENC_D_TRX_A
- R82 pad 2: Net-(U18-A) -> /TERM_A_R
- R83 pad 2: Net-(U19-A) -> /TERM_B_R
- R84 pad 2: Net-(U20-A) -> /TERM_C_R
- R85 pad 2: Net-(U21-A) -> /TERM_D_R
- U18 pad 6: Net-(U18-A) -> /ENC_A_TRX_A
- U19 pad 6: Net-(U19-A) -> /ENC_B_TRX_A
- U20 pad 6: Net-(U20-A) -> /ENC_C_TRX_A
- U21 pad 6: Net-(U21-A) -> /ENC_D_TRX_A
Routing:
- net +3V3: track 256.6 -> 204.2 mm, vias 17 -> 15
- net /ENC_D_N: track 36.0 -> 0.00 mm, vias 1 -> 0
- net /ENC_B_SW: track 110.8 -> 78.8 mm, vias 2 -> 1
- net /HALL3: track 93.8 -> 62.1 mm, vias 2 -> 1
- net /ENC_D_P: track 31.9 -> 1.70 mm, vias 1 -> 0
- net /V_ENC: track 34.0 -> 5.96 mm, vias 2 -> 1
- net /I2C_SDA: track 117.1 -> 89.2 mm, vias 5 -> 4
- net /H3_SW: track 95.8 -> 69.0 mm, vias 3 -> 2
- net GND: track 223.5 -> 198.2 mm, vias 238 -> 231
- net /ENC_A_SW: track 95.6 -> 70.5 mm, vias 3 -> 1
- net /HALL1: track 103.2 -> 80.2 mm, vias 3 -> 1
- net Vdrive: track 246.6 -> 224.1 mm
- net /HALL2: track 105.9 -> 84.9 mm, vias 2 -> 1
- net /EXT_ANALOG_SW: track 76.6 -> 55.8 mm, vias 3 -> 2
- net /EXT_ANALOG1: track 71.6 -> 51.3 mm, vias 2 -> 1
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
Commit message: Protection philosophy per design intent: 80V silicon, TVS just below
- Bridge FETs back to BSC030N08NS5 (80V, C501507) — the original part;
  60V bus on 80V silicon with TVS as the first line is the intended margin
  stack, not 100V FETs
- Bus TVS: SMDJ64A (standoff 64V > 60V bus, breakdown 71-79V < 80V FETs),
  matching the SMAJ64A phase TVS — every TVS now conducts before any FET
  avalanches
- README updated to state the philosophy and the rev-A ~48V limit

Netlist-verified: value-only change.

Co-Authored-By: Claude Fable 5 <noreply@anthropic.com>
Parts:
- AH1, AL1, BH1, BL1, CH1, CH2, CL1, CL2: value BSC040N10NS5 -> BSC030N08NS5
- D5: value SMDJ60A -> SMDJ64A
Changed lines of the file:
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@@
 			)
 		)
-		(property "Value" "BSC040N10NS5"
+		(property "Value" "BSC030N08NS5"
 			(at 0 3.5 90)
 			(layer "F.Fab")
@@
 			)
 		)
-		(property "LCSC" "LCSC-TBD-BSC040N10NS5"
+		(property "LCSC" "C501507"
 			(at 0 0 0)
 			(layer "F.Fab")
@@
 			)
 		)
-		(property "Value" "BSC040N10NS5"
+		(property "Value" "BSC030N08NS5"
 			(at 0 3.5 90)
 			(layer "F.Fab")
@@
 			)
 		)
-		(property "LCSC" "LCSC-TBD-BSC040N10NS5"
+		(property "LCSC" "C501507"
 			(at 0 0 0)
 			(layer "F.Fab")
@@
 			)
 		)
-		(property "Value" "BSC040N10NS5"
+		(property "Value" "BSC030N08NS5"
 			(at 0 3.5 0)
 			(layer "F.Fab")
@@
 			)
 		)
-		(property "LCSC" "LCSC-TBD-BSC040N10NS5"
+		(property "LCSC" "C501507"
 			(at 0 0 0)
 			(layer "F.Fab")
@@
 			)
 		)
-		(property "Value" "BSC040N10NS5"
+		(property "Value" "BSC030N08NS5"
 			(at 0 3.5 0)
 			(layer "F.Fab")
@@
 			)
 		)
-		(property "LCSC" "LCSC-TBD-BSC040N10NS5"
+		(property "LCSC" "C501507"
 			(at 0 0 0)
 			(layer "F.Fab")
@@
 			)
 		)
-		(property "Value" "BSC040N10NS5"
+		(property "Value" "BSC030N08NS5"
 			(at 0 3.5 90)
 			(layer "F.Fab")
@@
 			)
 		)
-		(property "LCSC" "LCSC-TBD-BSC040N10NS5"
+		(property "LCSC" "C501507"
 			(at 0 0 0)
 			(layer "F.Fab")
@@
 			)
 		)
-		(property "Value" "BSC040N10NS5"
+		(property "Value" "BSC030N08NS5"
 			(at 0 3.5 0)
 			(layer "F.Fab")
@@
 			)
 		)
-		(property "LCSC" "LCSC-TBD-BSC040N10NS5"
+		(property "LCSC" "C501507"
 			(at 0 0 0)
 			(layer "F.Fab")
@@
 			)
 		)
-		(property "Value" "BSC040N10NS5"
+		(property "Value" "BSC030N08NS5"
 			(at 0 3.5 90)
 			(layer "F.Fab")
@@
 			)
 		)
-		(property "LCSC" "LCSC-TBD-BSC040N10NS5"
+		(property "LCSC" "C501507"
 			(at 0 0 90)
 			(layer "F.Fab")
@@
 			)
 		)
-		(property "Value" "BSC040N10NS5"
+		(property "Value" "BSC030N08NS5"
 			(at 0 3.5 180)
 			(layer "F.Fab")
@@
 			)
 		)
-		(property "LCSC" "LCSC-TBD-BSC040N10NS5"
+		(property "LCSC" "C501507"
 			(at 0 0 0)
 			(layer "F.Fab")
@@
 			)
 		)
-		(property "Value" "SMDJ60A"
+		(property "Value" "SMDJ64A"
 			(at 0 -4.199999 0)
 			(layer "B.Fab")
@@
 			)
 		)
-		(property "LCSC" "LCSC-TBD-SMDJ60A"
+		(property "LCSC" "LCSC-TBD-SMDJ64A"
 			(at 0 0 0)
 			(layer "B.Fab")
