File: hardware/rp2350_driver.kicad_sch (KiCad schematic)
At the start: 291 parts, among them J1 XT30, J10 Power Output, J11 CAN2 PLUG, J12 Conn_01x06, J2 XT30, J3 USB_C_Receptacle_USB2.0, J4 SM03B-SRSS-TB, J5 Estop Conn, J6 SM03B-SRSS-TB, J7 Conn_01x03, J8 Conn_01x03, J9 XT30, Q1 Q_PNP_BEC, Q2 Q_PNP_BEC, Q3 Q_PNP_BEC, Q4 Q_PNP_BEC, Q5 Q_NMOS_GDS, SW1 Button, SW2 Button, U1 EG3113, U10 INA240A1D, U101 FUSB302BMPX, U11 USBLC6-2P6, U12 EG3113, U13 TS5A3159DCK, U14 TS5A3159DCK, U15 TS5A3159DCK, U16 CA-IS3052CG, U17 TS5A3159DCK, U18 SIT3088ETK, U19 SIT3088ETK, U20 SIT3088ETK, U21 SIT3088ETK, U22 TS5A3159DCK, U23 TS5A3159DCK, U24 TS5A3159DCK, U25 TS5A3159DCK, U26 TS5A3159DCK, U27 TS5A3159DCK, U28 XL7005A, U29 LM74700, U3 W25Q16JV, U4 SPX3819M5-L-3-3, U5 INA240A1D, U6 EG3113, U7 EG3113, U8 RP2350_80QFN, U9 INA240A1D, Y1 ABM8-272-T3

Commit message: Fix protection voltage ratings for real 60V operation
- FETs: BSC030N08NS5 (80V, C501507) -> TMG08N10SI (100V, C7422896); same
  PowerPAK SO-8 footprint, already vetted in the JLC cart
- Phase TVS D9/D13/D17/D21: SMAJ51A -> SMAJ64A. 51V standoff sat in
  leakage/breakdown whenever the bus exceeded ~51V with a high side on;
  64V standoff clears a 60V bus
- Bus TVS D5: SMDJ85A -> SMDJ60A. 85V standoff could never clamp before
  the old 80V FETs; 60V standoff clamps ~97V, inside the new FETs' 100V

LCSC numbers for the two new TVS values are marked LCSC-TBD — pick in-stock
parts at order time. Netlist-verified: value-only change, topology untouched.

Co-Authored-By: Claude Fable 5 <noreply@anthropic.com>
Parts:
- AH1, AL1, BH1, BL1, CH1, CH2, CL1, CL2: value MOSFETSO-8 -> TMG08N10SI; LCSC C501507 -> C7422896
- D13, D17, D21, D9: value SMAJ51A -> SMAJ64A; LCSC C366557 -> LCSC-TBD-SMAJ64A
- D5: value SMDJ85A -> SMDJ60A; LCSC C2990214 -> LCSC-TBD-SMDJ60A
Changed lines of the file:
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@@
 			)
 		)
-		(property "Value" "MOSFETSO-8"
+		(property "Value" "TMG08N10SI"
 			(at 110.998 426.974 0)
 			(effects
@@
 			)
 		)
-		(property "LCSC" "C501507"
+		(property "LCSC" "C7422896"
 			(at 119.38 420.37 0)
 			(effects
@@
 			)
 		)
-		(property "Value" "SMAJ51A"
+		(property "Value" "SMAJ64A"
 			(at 325.755 447.675 90)
 			(effects
@@
 			)
 		)
-		(property "LCSC" "C366557"
+		(property "LCSC" "LCSC-TBD-SMAJ64A"
 			(at 323.85 441.96 90)
 			(effects
@@
 			)
 		)
-		(property "Value" "MOSFETSO-8"
+		(property "Value" "TMG08N10SI"
 			(at 488.188 480.314 0)
 			(effects
@@
 			)
 		)
-		(property "LCSC" "C501507"
+		(property "LCSC" "C7422896"
 			(at 496.57 473.71 0)
 			(effects
@@
 			)
 		)
-		(property "Value" "MOSFETSO-8"
+		(property "Value" "TMG08N10SI"
 			(at 224.028 508.254 0)
 			(effects
@@
 			)
 		)
-		(property "LCSC" "C501507"
+		(property "LCSC" "C7422896"
 			(at 232.41 501.65 0)
 			(effects
@@
 			)
 		)
-		(property "Value" "MOSFETSO-8"
+		(property "Value" "TMG08N10SI"
 			(at 224.028 493.014 0)
 			(effects
@@
 			)
 		)
-		(property "LCSC" "C501507"
+		(property "LCSC" "C7422896"
 			(at 232.41 486.41 0)
 			(effects
@@
 			)
 		)
-		(property "Value" "MOSFETSO-8"
+		(property "Value" "TMG08N10SI"
 			(at 292.608 428.244 0)
 			(effects
@@
 			)
 		)
-		(property "LCSC" "C501507"
+		(property "LCSC" "C7422896"
 			(at 300.99 421.64 0)
 			(effects
@@
 			)
 		)
-		(property "Value" "SMAJ51A"
+		(property "Value" "SMAJ64A"
 			(at 511.175 484.505 90)
 			(effects
@@
 			)
 		)
-		(property "LCSC" "C366557"
+		(property "LCSC" "LCSC-TBD-SMAJ64A"
 			(at 509.27 478.79 90)
 			(effects
@@
 			)
 		)
-		(property "Value" "MOSFETSO-8"
+		(property "Value" "TMG08N10SI"
 			(at 119.888 442.214 0)
 			(effects
@@
 			)
 		)
-		(property "LCSC" "C501507"
+		(property "LCSC" "C7422896"
 			(at 128.27 435.61 0)
 			(effects
@@
 			)
 		)
-		(property "Value" "SMAJ51A"
+		(property "Value" "SMAJ64A"
 			(at 144.78 445.77 90)
 			(effects
@@
 			)
 		)
-		(property "LCSC" "C366557"
+		(property "LCSC" "LCSC-TBD-SMAJ64A"
 			(at 143.51 439.42 90)
 			(effects
@@
 			)
 		)
-		(property "Value" "MOSFETSO-8"
+		(property "Value" "TMG08N10SI"
 			(at 478.028 465.074 0)
 			(effects
@@
 			)
 		)
-		(property "LCSC" "C501507"
+		(property "LCSC" "C7422896"
 			(at 486.41 458.47 0)
 			(effects
@@
 			)
 		)
-		(property "Value" "SMAJ51A"
+		(property "Value" "SMAJ64A"
 			(at 248.285 509.27 90)
 			(effects
@@
 			)
 		)
-		(property "LCSC" "C366557"
+		(property "LCSC" "LCSC-TBD-SMAJ64A"
 			(at 246.38 506.73 90)
 			(effects
@@
 			)
 		)
-		(property "Value" "SMDJ85A"
+		(property "Value" "SMDJ60A"
 			(at 101.6 485.775 90)
 			(effects
@@
 			)
 		)
-		(property "LCSC" "C2990214"
+		(property "LCSC" "LCSC-TBD-SMDJ60A"
 			(at 99.06 483.87 90)
 			(effects
@@
 			)
 		)
-		(property "Value" "MOSFETSO-8"
+		(property "Value" "TMG08N10SI"
 			(at 302.768 443.484 0)
 			(effects
@@
 			)
 		)
-		(property "LCSC" "C501507"
+		(property "LCSC" "C7422896"
 			(at 311.15 436.88 0)
 			(effects

Commit message: Add switched RS-485 termination + P-line pull-ups to encoder port
Fixes single-ended encoder support: the fixed 100R terminations R82-R85
coupled the undriven line to the driven one 50:1 against the 10k/10k bias,
so a single-ended signal only developed +/-32mV of differential -- below
the SIT3088's -200..-100mV threshold. Termination is now in series with a
TS5A3159 per channel (U30-U33), all enabled by TERM_SW = GPIO38 (which was
already routed to TP20, so current boards can be bodged):

  TERM_SW high -> 100R in circuit (differential encoders)
  TERM_SW low / boot default -> open; B input rests at the 1.65V bias and
  single-ended signals see +/-1.65V of differential

R97-R100 (10k to 3V3) pull the P lines up so open-collector encoders work
too; C110-C113 decouple the new switches. R82-R85 moved beside their
switches; transceiver-side nets now labeled ENC_x_TRX_A/B.

Netlist-verified: only the intended nodes changed. ERC delta is 16 benign
lib-drift warnings of the kind the sheet already carries.

Co-Authored-By: Claude Fable 5 <noreply@anthropic.com>
Parts:
- added C110, C111, C112, C113: 100n, Capacitor_SMD:C_0402_1005Metric, symbol Device:C
- added R100, R97, R98, R99: 10k, Resistor_SMD:R_0402_1005Metric, symbol Device:R
- added U30, U31, U32, U33: TS5A3159DCK, Package_TO_SOT_SMD:SOT-363_SC-70-6, symbol integrated:TS5A3159
Connections:
- net +3V3: now also R100.1, R97.1, R98.1, R99.1
- net ENC_A_P_SW: now also R97.2
- net ENC_B_P_SW: now also R98.2
- net ENC_C_P_SW: now also R99.2
- net ENC_D_P: now also R100.2
- net GND: now also C110.2, C111.2, C112.2, C113.2, U30.2 (GND), U31.2 (GND), U32.2 (GND), U33.2 (GND)
- net Vdrive: now also C110.1, C111.1, C112.1, C113.1, U30.5 (V+), U31.5 (V+), U32.5 (V+), U33.5 (V+)
- net ENC_B_TRX_B: now reaches FL1.1, U19.7 (B)
- net ENC_B_TRX_B: now also R83.2; no longer R83.1
- net ENC_B_TRX_A: now reaches FL1.4, U19.6 (A)
- net ENC_B_TRX_A: now also U31.4 (COM); no longer R83.2
- net ENC_D_TRX_B: now reaches FL4.1, U21.7 (B)
- net ENC_D_TRX_B: now also R85.2; no longer R85.1
- net ENC_D_TRX_A: now reaches FL4.4, U21.6 (A)
- net ENC_D_TRX_A: now also U33.4 (COM); no longer R85.2
- net ENC_A_TRX_A: now reaches FL2.4, U18.6 (A)
- net ENC_A_TRX_A: now also U30.4 (COM); no longer R82.2
- net ENC_A_TRX_B: now reaches FL2.1, U18.7 (B)
- net ENC_A_TRX_B: now also R82.2; no longer R82.1
- net TERM_SW: now reaches TP20.1, U8.47 (GPIO38)
- net TERM_SW: now also U30.6 (ENB), U31.6 (ENB), U32.6 (ENB), U33.6 (ENB)
- net ENC_C_TRX_B: now reaches FL3.1, U20.7 (B)
- net ENC_C_TRX_B: now also R84.2; no longer R84.1
- net ENC_C_TRX_A: now reaches FL3.4, U20.6 (A)
- net ENC_C_TRX_A: now also U32.4 (COM); no longer R84.2
- new net TERM_A_R: R82.1, U30.1 (NO)
- new net TERM_B_R: R83.1, U31.1 (NO)
- new net TERM_C_R: R84.1, U32.1 (NO)
- new net TERM_D_R: R85.1, U33.1 (NO)
- no-connect marks 0 -> 4
Other:
- note added: "Rev B: switchable RS-485 termination. TERM_SW (GPIO38/TP20) high = 100R termination in circuit (differential encoders). Low/boot default = termination open: single-ended signals see the 10k/10k bias as a 1.65V threshold. R97-R100 pull P lines up for open-collector encoders."
- moved on the sheet: R82, R83, R84, R85

Commit message: Define boot states, fix WS2812 logic margin, add DNP hardware E-stop
- R101-R112: 100k pull-downs on every TS5A3159 enable and SIT3088 DE/RE
  line (V_SW, I2C_SW, H1-3_SW, EXT_ANALOG_SW, TH_SW_1, ENC_A-D_SW,
  TERM_SW). These all floated between power-up and firmware init; worst
  case V_SW could select 5V onto a 3.3V encoder. Defaults are now:
  V_ENC=3.3V, transceivers receiving, alternate paths off, termination open
- D30 (DSS110) + C114: WS2812 now runs from LED_VDD = Vdrive minus one
  Schottky drop, so 3.3V data satisfies VIH = 0.7*VDD (was 3.5V at 5.0V)
- Q6 + R113 (both DNP): populate to make an open E-stop loop pull RUN low,
  braking the motor via the gate-driver input pulls with no firmware in
  the loop. Unpopulated boards keep today's GPIO-only behavior

Netlist-verified node-for-node; ERC delta is lib-drift warnings only.

Co-Authored-By: Claude Fable 5 <noreply@anthropic.com>
Parts:
- added C114: 100n, Capacitor_SMD:C_0402_1005Metric, symbol Device:C
- added D30: DSS110, Diode_SMD:D_SOD-123F, symbol Device:D
- added Q6: 2N7002, Package_TO_SOT_SMD:SOT-23, symbol Transistor_FET:Q_NMOS_GDS
- added R101, R102, R103, R104, R105, R106, R107, R108, R109, R110, R111, R112: 100k, Resistor_SMD:R_0402_1005Metric, symbol Device:R
- added R113: 10k, Resistor_SMD:R_0402_1005Metric, symbol Device:R
Connections:
- net +3V3: now also R113.1
- net E-STOP: now also Q6.1 (G), R113.2
- net ENC_A_SW: now also R108.1
- net ENC_B_SW: now also R109.1
- net ENC_C_SW: now also R110.1
- net ENC_D_SW: now also R111.1
- net EXT_ANALOG_SW: now also R106.1
- net GND: now also C114.2, Q6.3 (S), R101.2, R102.2, R103.2, R104.2, R105.2, R106.2, R107.2, R108.2, R109.2, R110.2, R111.2, R112.2
- net H1_SW: now also R103.1
- net H2_SW: now also R104.1
- net H3_SW: now also R105.1
- net I2C_SW: now also R102.1
- net RUN: now also Q6.2 (D)
- net TERM_SW: now also R112.1
- net TH_SW_1: now also R107.1
- net V_SW: now also R101.1
- net Vdrive: now also D30.2 (A); no longer D1.3 (VDD)
- new net LED_VDD: C114.1, D1.3 (VDD), D30.1 (K)
Other:
- note added: "DNP option: hardware E-stop. Populate Q6 + R113 and an open E-stop loop resets the CPU (RUN low) -> gate-driver pulls brake the motor with no firmware in the loop. Unpopulated = current GPIO-only behavior."
- note added: "Rev B: defined boot states. 100k pull-downs: every analog-switch enable + transceiver DE/RE floats between power-up and firmware init. Defaults: V_ENC=3.3V, transceivers in receive, hall/I2C/analog paths off, termination open."
- note added: "WS2812 runs from LED_VDD = Vdrive - one Schottky drop (~4.5V), so 3.3V data meets VIH = 0.7*VDD with margin."

Commit message: Correct bridge FET part; map R82-R85 pins to preserve existing copper
- Bridge FETs: TMG08N10SI was wrong -- C7422896 is the SOT-89 FET already
  used at Q5 (LM74700 ideal diode), not a PowerPAK part. Bridge is now
  BSC040N10NS5 (Infineon OptiMOS 100V, PowerPAK SO-8), LCSC marked TBD for
  verification at order time
- R82-R85 pin1 now stays on the transceiver B line (its existing PCB stub
  is untouched); only pin2 moves to the new TERM_x_R switch net, so the
  board edit is a single cut per channel

Co-Authored-By: Claude Fable 5 <noreply@anthropic.com>
Parts:
- AH1, AL1, BH1, BL1, CH1, CH2, CL1, CL2: value TMG08N10SI -> BSC040N10NS5; LCSC C7422896 -> LCSC-TBD-BSC040N10NS5
Connections:
- net ENC_A_TRX_B: now also R82.1; no longer R82.2
- net ENC_B_TRX_B: now also R83.1; no longer R83.2
- net ENC_C_TRX_B: now also R84.1; no longer R84.2
- net ENC_D_TRX_B: now also R85.1; no longer R85.2
- net TERM_A_R: now also R82.2; no longer R82.1
- net TERM_B_R: now also R83.2; no longer R83.1
- net TERM_C_R: now also R84.2; no longer R84.1
- net TERM_D_R: now also R85.2; no longer R85.1
Changed lines of the file:
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@@
 			)
 		)
-		(property "Value" "TMG08N10SI"
+		(property "Value" "BSC040N10NS5"
 			(at 110.998 426.974 0)
 			(effects
@@
 			)
 		)
-		(property "LCSC" "C7422896"
+		(property "LCSC" "LCSC-TBD-BSC040N10NS5"
 			(at 119.38 420.37 0)
 			(effects
@@
 			)
 		)
-		(property "Value" "TMG08N10SI"
+		(property "Value" "BSC040N10NS5"
 			(at 488.188 480.314 0)
 			(effects
@@
 			)
 		)
-		(property "LCSC" "C7422896"
+		(property "LCSC" "LCSC-TBD-BSC040N10NS5"
 			(at 496.57 473.71 0)
 			(effects
@@
 			)
 		)
-		(property "Value" "TMG08N10SI"
+		(property "Value" "BSC040N10NS5"
 			(at 224.028 508.254 0)
 			(effects
@@
 			)
 		)
-		(property "LCSC" "C7422896"
+		(property "LCSC" "LCSC-TBD-BSC040N10NS5"
 			(at 232.41 501.65 0)
 			(effects
@@
 			)
 		)
-		(property "Value" "TMG08N10SI"
+		(property "Value" "BSC040N10NS5"
 			(at 224.028 493.014 0)
 			(effects
@@
 			)
 		)
-		(property "LCSC" "C7422896"
+		(property "LCSC" "LCSC-TBD-BSC040N10NS5"
 			(at 232.41 486.41 0)
 			(effects
@@
 			)
 		)
-		(property "Value" "TMG08N10SI"
+		(property "Value" "BSC040N10NS5"
 			(at 292.608 428.244 0)
 			(effects
@@
 			)
 		)
-		(property "LCSC" "C7422896"
+		(property "LCSC" "LCSC-TBD-BSC040N10NS5"
 			(at 300.99 421.64 0)
 			(effects
@@
 			)
 		)
-		(property "Value" "TMG08N10SI"
+		(property "Value" "BSC040N10NS5"
 			(at 119.888 442.214 0)
 			(effects
@@
 			)
 		)
-		(property "LCSC" "C7422896"
+		(property "LCSC" "LCSC-TBD-BSC040N10NS5"
 			(at 128.27 435.61 0)
 			(effects
@@
 			)
 		)
-		(property "Value" "TMG08N10SI"
+		(property "Value" "BSC040N10NS5"
 			(at 478.028 465.074 0)
 			(effects
@@
 			)
 		)
-		(property "LCSC" "C7422896"
+		(property "LCSC" "LCSC-TBD-BSC040N10NS5"
 			(at 486.41 458.47 0)
 			(effects
@@
 			)
 		)
-		(property "Value" "TMG08N10SI"
+		(property "Value" "BSC040N10NS5"
 			(at 302.768 443.484 0)
 			(effects
@@
 			)
 		)
-		(property "LCSC" "C7422896"
+		(property "LCSC" "LCSC-TBD-BSC040N10NS5"
 			(at 311.15 436.88 0)
 			(effects
@@
 		)
 	)
-	(label "TERM_A_R"
+	(label "ENC_A_TRX_B"
 		(at 708.6600000000001 511.81 0)
 		(effects
@@
 		)
 	)
-	(label "ENC_A_TRX_B"
+	(label "TERM_A_R"
 		(at 708.6600000000001 521.97 0)
 		(effects
@@
 		)
 	)
-	(label "TERM_B_R"
+	(label "ENC_B_TRX_B"
 		(at 742.95 511.81 0)
 		(effects
@@
 		)
 	)
-	(label "ENC_B_TRX_B"
+	(label "TERM_B_R"
 		(at 742.95 521.97 0)
 		(effects
@@
 		)
 	)
-	(label "TERM_C_R"
+	(label "ENC_C_TRX_B"
 		(at 777.2400000000001 511.81 0)
 		(effects
@@
 		)
 	)
-	(label "ENC_C_TRX_B"
+	(label "TERM_C_R"
 		(at 777.2400000000001 521.97 0)
 		(effects
@@
 		)
 	)
-	(label "TERM_D_R"
+	(label "ENC_D_TRX_B"
 		(at 811.5300000000001 511.81 0)
 		(effects
@@
 		)
 	)
-	(label "ENC_D_TRX_B"
+	(label "TERM_D_R"
 		(at 811.5300000000001 521.97 0)
 		(effects

Commit message: Protection philosophy per design intent: 80V silicon, TVS just below
- Bridge FETs back to BSC030N08NS5 (80V, C501507) — the original part;
  60V bus on 80V silicon with TVS as the first line is the intended margin
  stack, not 100V FETs
- Bus TVS: SMDJ64A (standoff 64V > 60V bus, breakdown 71-79V < 80V FETs),
  matching the SMAJ64A phase TVS — every TVS now conducts before any FET
  avalanches
- README updated to state the philosophy and the rev-A ~48V limit

Netlist-verified: value-only change.

Co-Authored-By: Claude Fable 5 <noreply@anthropic.com>
Parts:
- AH1, AL1, BH1, BL1, CH1, CH2, CL1, CL2: value BSC040N10NS5 -> BSC030N08NS5; LCSC LCSC-TBD-BSC040N10NS5 -> C501507
- D5: value SMDJ60A -> SMDJ64A; LCSC LCSC-TBD-SMDJ60A -> LCSC-TBD-SMDJ64A
Changed lines of the file:
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@@
 			)
 		)
-		(property "Value" "BSC040N10NS5"
+		(property "Value" "BSC030N08NS5"
 			(at 110.998 426.974 0)
 			(effects
@@
 			)
 		)
-		(property "LCSC" "LCSC-TBD-BSC040N10NS5"
+		(property "LCSC" "C501507"
 			(at 119.38 420.37 0)
 			(effects
@@
 			)
 		)
-		(property "Value" "BSC040N10NS5"
+		(property "Value" "BSC030N08NS5"
 			(at 488.188 480.314 0)
 			(effects
@@
 			)
 		)
-		(property "LCSC" "LCSC-TBD-BSC040N10NS5"
+		(property "LCSC" "C501507"
 			(at 496.57 473.71 0)
 			(effects
@@
 			)
 		)
-		(property "Value" "BSC040N10NS5"
+		(property "Value" "BSC030N08NS5"
 			(at 224.028 508.254 0)
 			(effects
@@
 			)
 		)
-		(property "LCSC" "LCSC-TBD-BSC040N10NS5"
+		(property "LCSC" "C501507"
 			(at 232.41 501.65 0)
 			(effects
@@
 			)
 		)
-		(property "Value" "BSC040N10NS5"
+		(property "Value" "BSC030N08NS5"
 			(at 224.028 493.014 0)
 			(effects
@@
 			)
 		)
-		(property "LCSC" "LCSC-TBD-BSC040N10NS5"
+		(property "LCSC" "C501507"
 			(at 232.41 486.41 0)
 			(effects
@@
 			)
 		)
-		(property "Value" "BSC040N10NS5"
+		(property "Value" "BSC030N08NS5"
 			(at 292.608 428.244 0)
 			(effects
@@
 			)
 		)
-		(property "LCSC" "LCSC-TBD-BSC040N10NS5"
+		(property "LCSC" "C501507"
 			(at 300.99 421.64 0)
 			(effects
@@
 			)
 		)
-		(property "Value" "BSC040N10NS5"
+		(property "Value" "BSC030N08NS5"
 			(at 119.888 442.214 0)
 			(effects
@@
 			)
 		)
-		(property "LCSC" "LCSC-TBD-BSC040N10NS5"
+		(property "LCSC" "C501507"
 			(at 128.27 435.61 0)
 			(effects
@@
 			)
 		)
-		(property "Value" "BSC040N10NS5"
+		(property "Value" "BSC030N08NS5"
 			(at 478.028 465.074 0)
 			(effects
@@
 			)
 		)
-		(property "LCSC" "LCSC-TBD-BSC040N10NS5"
+		(property "LCSC" "C501507"
 			(at 486.41 458.47 0)
 			(effects
@@
 			)
 		)
-		(property "Value" "SMDJ60A"
+		(property "Value" "SMDJ64A"
 			(at 101.6 485.775 90)
 			(effects
@@
 			)
 		)
-		(property "LCSC" "LCSC-TBD-SMDJ60A"
+		(property "LCSC" "LCSC-TBD-SMDJ64A"
 			(at 99.06 483.87 90)
 			(effects
@@
 			)
 		)
-		(property "Value" "BSC040N10NS5"
+		(property "Value" "BSC030N08NS5"
 			(at 302.768 443.484 0)
 			(effects
@@
 			)
 		)
-		(property "LCSC" "LCSC-TBD-BSC040N10NS5"
+		(property "LCSC" "C501507"
 			(at 311.15 436.88 0)
 			(effects
