File: hardware/rp2350_driver.kicad_sch (KiCad schematic)
At the start: 291 parts, among them J1 XT30, J10 Power Output, J11 CAN2 PLUG, J12 Conn_01x06, J2 XT30, J3 USB_C_Receptacle_USB2.0, J4 SM03B-SRSS-TB, J5 Estop Conn, J6 SM03B-SRSS-TB, J7 Conn_01x03, J8 Conn_01x03, J9 XT30, Q1 Q_PNP_BEC, Q2 Q_PNP_BEC, Q3 Q_PNP_BEC, Q4 Q_PNP_BEC, Q5 Q_NMOS_GDS, SW1 Button, SW2 Button, U1 EG3113, U10 INA240A1D, U101 FUSB302BMPX, U11 USBLC6-2P6, U12 EG3113, U13 TS5A3159DCK, U14 TS5A3159DCK, U15 TS5A3159DCK, U16 CA-IS3052CG, U17 TS5A3159DCK, U18 SIT3088ETK, U19 SIT3088ETK, U20 SIT3088ETK, U21 SIT3088ETK, U22 TS5A3159DCK, U23 TS5A3159DCK, U24 TS5A3159DCK, U25 TS5A3159DCK, U26 TS5A3159DCK, U27 TS5A3159DCK, U28 XL7005A, U29 LM74700, U3 W25Q16JV, U4 SPX3819M5-L-3-3, U5 INA240A1D, U6 EG3113, U7 EG3113, U8 RP2350_80QFN, U9 INA240A1D, Y1 ABM8-272-T3

Commit message: schematic: the rev-B schematic on the rev-A base, plus Tier A footprints
rp2350_driver.kicad_sch is rev-b-fixes @ ed7808b verbatim (F-19 CAN
termination, F-27/F-39 LTC4359 + Q5 PowerPAK + D31 + U11 pin 5, switched
encoder termination U30-U33 with pull-ups/downs, DNP E-stop Q6/R113,
LED_VDD drop diode D30, 80 V FETs and 64 V TVS values, F-43 0402 shrink),
then edit_sch_footprints.py re-pointed 208 Footprint fields:

  A1  snubbers R17 R18 R37 R38 R48 R52 R80 R81 -> R_0603_JLC,
      C7 C9 C25 C26 C33 C34 C53 C54 -> C_0402_JLC
  A2  TP12-TP20 -> TestPoint_Pad_D1.0mm_no_courtyard (pad size kept),
      TP8 Keystone loop -> TestPoint_Pad_D1.5mm_no_courtyard
  A3  all 14 TS5A3159DCK -> parts:SOT-363_SC-70-6_JLC
  A4  every R/C 0402/0603/0805 -> parts:*_JLC
  A5  D1 -> LED_WS2812B-2020 (MotorBuck pin order)

Netlist-verified against rev-b-fixes: components, values, DNP flags and
every pin-to-net identical; only footprint fields differ.

Co-Authored-By: Claude Fable 5.1 <noreply@anthropic.com>
Claude-Session: https://claude.ai/code/session_014kYruXdHPn5HC6gTNK16no
Parts:
- removed C79: 100n, Capacitor_SMD:C_0402_1005Metric, symbol Device:C
- added C110, C111, C112, C113, C114: 100n, parts:C_0402_1005Metric_JLC, symbol Device:C
- added C115: 1n 2kV, Capacitor_SMD:C_1206_3216Metric, symbol Device:C
- added D30: DSS110, Diode_SMD:D_SOD-123F, symbol Device:D
- added D31: SMF24A, Diode_SMD:D_SOD-123F, symbol Diode:SMAJ24A
- added JP2: Jumper_2_Open, Jumper:SolderJumper-2_P1.3mm_Open_RoundedPad1.0x1.5mm, symbol Jumper:Jumper_2_Open
- added Q6: 2N7002, Package_TO_SOT_SMD:SOT-23, symbol Transistor_FET:Q_NMOS_GDS
- added R100, R113, R97, R98, R99: 10k, parts:R_0402_1005Metric_JLC, symbol Device:R
- added R101, R102, R103, R104, R105, R106, R107, R108, R109, R110, R111, R112: 100k, parts:R_0402_1005Metric_JLC, symbol Device:R
- added R114: 120R, Resistor_SMD:R_0603_1608Metric, symbol Device:R
- added R115: 100R, Resistor_SMD:R_0603_1608Metric, symbol Device:R
- added U30, U31, U32, U33: TS5A3159DCK, parts:SOT-363_SC-70-6_JLC, symbol integrated:TS5A3159
- AH1, AL1, BH1, BL1, CH1, CH2, CL1, CL2: value MOSFETSO-8 -> BSC030N08NS5
- C10, C15, C2, C23, C27, C28, C31, C36, C48, C51, C55, C57, C58, C6, C69, C70, C75, C78, C81: footprint Capacitor_SMD:C_0603_1608Metric -> parts:C_0603_1608Metric_JLC
- C105, C106, C12, C47, C5: footprint Capacitor_SMD:C_0805_2012Metric -> parts:C_0805_2012Metric_JLC
- C107, C108, C13, C14, C20, C21, C22, C24, C3, C30, C32, C35, C37, C38, C4, C41, C43, C45, C46, C49, C50, C52, C56, C59, C60, C61, C62, C63, C64, C65, C66, C67, C68, C71, C72, C73, C74, C76, C77: footprint Capacitor_SMD:C_0402_1005Metric -> parts:C_0402_1005Metric_JLC
- C16, C19, C29, C40: footprint Capacitor_SMD:C_0603_1608Metric -> parts:C_0402_1005Metric_JLC
- C25, C26, C33, C34, C53, C54, C7, C9: footprint Capacitor_SMD:C_0805_2012Metric -> parts:C_0402_1005Metric_JLC
- D1: footprint RP2040_minimal:LED_WS2812_3528_3.5x2.8mm_P1.5mm -> parts:LED_WS2812B-2020_PLCC4_2.0x2.0mm_MotorBuck
- D13, D17, D21, D9: value SMAJ51A -> SMAJ64A; LCSC C366557 -> LCSC-TBD-SMAJ64A
- D5: value SMDJ85A -> SMDJ64A; LCSC C2990214 -> LCSC-TBD-SMDJ64A
- Q5: value Q_NMOS_GDS -> E100N4P0HL1; footprint Package_TO_SOT_SMD:SOT-89-3 -> parts:PowerPAK_SO-8_123; symbol Transistor_FET:Q_NMOS_GDS -> Device:Q_NMOS_SGD; LCSC C7422896 -> C29781176
- R1, R2, R21, R22, R35, R36, R49, R53, R54, R65, R66: footprint Resistor_SMD:R_0603_1608Metric -> parts:R_0402_1005Metric_JLC
- R10, R11, R12, R13, R14, R15, R25, R27, R28, R29, R30, R31, R33, R41, R42, R43, R44, R45, R46, R47, R59, R60, R61, R62, R63, R64, R67, R68, R69, R70, R71, R72, R73, R74, R75, R76, R77, R78, R79, R9, TH1: footprint Resistor_SMD:R_0603_1608Metric -> parts:R_0603_1608Metric_JLC
- R17, R18, R37, R38, R48, R52, R80, R81: footprint Resistor_SMD:R_0805_2012Metric -> parts:R_0603_1608Metric_JLC
- R24, R26, R32, R34, R5, R50, R51, R57, R58, R6, R8, R82, R83, R84, R85, R86, R87, R88, R89, R90, R91, R92, R93, R94, R95, R96: footprint Resistor_SMD:R_0402_1005Metric -> parts:R_0402_1005Metric_JLC
- TP12, TP13, TP14, TP15, TP16, TP17, TP18, TP19, TP20: footprint TestPoint:TestPoint_Pad_D1.0mm -> parts:TestPoint_Pad_D1.0mm_no_courtyard
- TP8: footprint TestPoint:TestPoint_Keystone_5019_Minature -> parts:TestPoint_Pad_D1.5mm_no_courtyard
- U13, U14, U15, U17, U22, U23, U24, U25, U26, U27: footprint Package_TO_SOT_SMD:SOT-363_SC-70-6 -> parts:SOT-363_SC-70-6_JLC
- U29: value LM74700 -> LTC4359CMS8; footprint Package_TO_SOT_SMD:SOT-23-6 -> Package_SO:MSOP-8_3x3mm_P0.65mm; symbol Power_Management:LM74700 -> Power_Management:LTC4359-MS8; LCSC C2941042 -> C688235
Connections:
- net +3V3: now also U11.5 (VBUS), R100.1, R113.1, R97.1, R98.1, R99.1
- net CAN0_N: now also JP2.2 (B)
- net CAN0_P: now also R114.1
- net E-STOP: now also Q6.1 (G), R113.2
- net ENC_A_P_SW: now also R97.2
- net ENC_A_SW: now also R108.1
- net ENC_B_P_SW: now also R98.2
- net ENC_B_SW: now also R109.1
- net ENC_C_P_SW: now also R99.2
- net ENC_C_SW: now also R110.1
- net ENC_D_P: now also R100.2
- net ENC_D_SW: now also R111.1
- net EXT_ANALOG_SW: now also R106.1
- net GND: now also U29.6 (Vss), C110.2, C111.2, C112.2, C113.2, C114.2, D31.2 (A2), Q6.3 (S), R101.2, R102.2, R103.2, R104.2, R105.2, R106.2, R107.2, R108.2, R109.2, R110.2, R111.2, R112.2, R115.2, U30.2 (GND), U31.2 (GND), U32.2 (GND), U33.2 (GND); no longer U29.2 (GND)
- net GND_ISO: now also C115.1
- net H1_SW: now also R103.1
- net H2_SW: now also R104.1
- net H3_SW: now also R105.1
- net I2C_SW: now also R102.1
- net RUN: now also Q6.2 (D)
- net TH_SW_1: now also R107.1
- net VBUS: now also Q5.1 (S), U29.2 (SRC), U29.4 (IN), U29.5 (~{SHDN}), D31.1 (A1); no longer Q5.3 (S), U11.5 (VBUS), U29.3 (EN), U29.6 (ANODE)
- net V_SW: now also R101.1
- net Vdrive: now also C110.1, C111.1, C112.1, C113.1, D30.2 (A), U30.5 (V+), U31.5 (V+), U32.5 (V+), U33.5 (V+); no longer D1.3 (VDD)
- net ENC_B_TRX_B: now reaches FL1.1, R83.1, U19.7 (B)
- net ENC_B_TRX_A: now reaches FL1.4, U19.6 (A)
- net ENC_B_TRX_A: now also U31.4 (COM); no longer R83.2
- net at C78.2, JP1.1 (A): now also Q5.3 (D), U29.8 (OUT); no longer Q5.2 (D), U29.4 (CATHODE)
- net ENC_D_TRX_B: now reaches FL4.1, R85.1, U21.7 (B)
- net ENC_D_TRX_A: now reaches FL4.4, U21.6 (A)
- net ENC_D_TRX_A: now also U33.4 (COM); no longer R85.2
- net ENC_A_TRX_A: now reaches FL2.4, U18.6 (A)
- net ENC_A_TRX_A: now also U30.4 (COM); no longer R82.2
- net ENC_A_TRX_B: now reaches FL2.1, R82.1, U18.7 (B)
- net TERM_SW: now reaches TP20.1, U8.47 (GPIO38)
- net TERM_SW: now also R112.1, U30.6 (ENB), U31.6 (ENB), U32.6 (ENB), U33.6 (ENB)
- net at U29.1 (GATE): now also Q5.2 (G)
- net ENC_C_TRX_B: now reaches FL3.1, R84.1, U20.7 (B)
- net ENC_C_TRX_A: now reaches FL3.4, U20.6 (A)
- net ENC_C_TRX_A: now also U32.4 (COM); no longer R84.2
- new net: C115.2, R115.1
- new net: JP2.1 (A), R114.2
- new net LED_VDD: C114.1, D1.3 (VDD), D30.1 (K)
- new net TERM_A_R: R82.2, U30.1 (NO)
- new net TERM_B_R: R83.2, U31.1 (NO)
- new net TERM_C_R: R84.2, U32.1 (NO)
- new net TERM_D_R: R85.2, U33.1 (NO)
- no-connect marks 0 -> 4
Other:
- note added: "DNP option: hardware E-stop. Populate Q6 + R113 and an open E-stop loop resets the CPU (RUN low) -> gate-driver pulls brake the motor with no firmware in the loop. Unpopulated = current GPIO-only behavior."
- note added: "F-19 (a): end-of-bus termination. JP2 open = un-terminated, the shipping default for a mid-bus node. Bridge JP2 to put R114 (120R) across CANH/CANL when this board sits at a bus end. Termination is on the isolated side, so it is powered by the harness like U16."
- note added: "F-19 (b): isolation-barrier stitch. GND_ISO is powered and referenced ONLY by the CAN harness (J11) -- no board 5V/GND feeds the isolated side, so isolation depends on the harness supplying +5V_ISO. C115 blocks DC so the barrier holds, while giving common-mode current a defined return instead of letting it radiate off the harness. R115 damps the C115/trace resonance and limits surge current. LAYO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"
- note added: "Rev B: defined boot states. 100k pull-downs: every analog-switch enable + transceiver DE/RE floats between power-up and firmware init. Defaults: V_ENC=3.3V, transceivers in receive, hall/I2C/analog paths off, termination open."
- note added: "Rev B: switchable RS-485 termination. TERM_SW (GPIO38/TP20) high = 100R termination in circuit (differential encoders). Low/boot default = termination open: single-ended signals see the 10k/10k bias as a 1.65V threshold. R97-R100 pull P lines up for open-collector encoders."
- note added: "WS2812 runs from LED_VDD = Vdrive - one Schottky drop (~4.5V), so 3.3V data meets VIH = 0.7*VDD with margin."
- moved on the sheet: R82, R83, R84, R85, U29
