File: hardware/tools/settle/candidates/plan_of_record.kicad_pcb (KiCad board)
At the start: 6 copper layers, 76 x 46.4 mm, 323 parts, among them J1 XT30, J10 Power Output, J11 CAN2 PLUG, J12 Conn_01x06, J2 XT30, J3 USB_C_Receptacle_USB2.0, J4 SM03B-SRSS-TB, J5 Estop Conn, J6 SM03B-SRSS-TB, J7 Conn_01x03, J8 Conn_01x03, J9 XT30, Q1 Q_PNP_BEC, Q2 Q_PNP_BEC, Q3 Q_PNP_BEC, Q4 Q_PNP_BEC, Q5 E100N4P0HL1, Q6 2N7002, SW1 Button, SW2 Button, U1 EG3113, U10 INA240A1D, U101 FUSB302BMPX, U11 USBLC6-2P6, U12 EG3113, U13 TS5A3159DCK, U14 TS5A3159DCK, U15 TS5A3159DCK, U16 CA-IS3052CG, U17 TS5A3159DCK, U18 SIT3088ETK, U19 SIT3088ETK, U20 SIT3088ETK, U21 SIT3088ETK, U22 TS5A3159DCK, U23 TS5A3159DCK, U24 TS5A3159DCK, U25 TS5A3159DCK, U26 TS5A3159DCK, U27 TS5A3159DCK, U28 XL7005A, U29 LTC4359CMS8, U3 W25Q16JV, U30 TS5A3159DCK, U31 TS5A3159DCK, U32 TS5A3159DCK, U33 TS5A3159DCK, U4 SPX3819M5-L-3-3, U5 INA240A1D, U6 EG3113, U7 EG3113, U8 RP2350_80QFN, U9 INA240A1D, Y1 ABM8-272-T3

Commit message: settle: mounting-hole keepouts on the plan of record, six pulldowns out of the rings
The edge half-hole footprint (parts:MountingHole_3.9mm_Plastite_#6) had
a top-only 3.65 mm courtyard and no rule area, so the settle engine left
six rev-B pulldowns under the screw heads. The footprint now carries a
rule area on F.Cu + B.Cu (no tracks, no footprints; vias, pads and pours
allowed) and the missing B.CrtYd circle.

On the candidate board: R105 R106 R109 R111 R112 R113 moved to searched
free spots; C5, C12, U10 and the R56/R55/D17 column nudged 0.05-0.35 mm
with track ends dragged; the +3V3 link to U10 that hugged H3 on B.Cu
moved to In3; I2C_SDA lifted off H2. kicad-cli DRC: keepout violations
20 -> 0, courtyard errors at baseline, 103 airwires unchanged.

Only the candidate is fixed. The same pulldowns still sit inside the
rings on rev-b-fixes, rev-b-lean and this branch's rp2350_driver board.
Written up in review/renders.html#keepouts.

Co-Authored-By: Claude Opus 5.5 <noreply@anthropic.com>
Parts:
- moved R109 6.53 mm to (124.6, 85.8), turned to 0 degrees
- moved R106 4.18 mm to (134.0, 126.1), turned to 90 degrees
- moved R111 3.64 mm to (180.5, 124.8), turned to 0 degrees
- moved R112 3.16 mm to (179.1, 86.3), turned to 0 degrees
- moved R105 2.06 mm to (135.1, 126.2), turned to -90 degrees
- moved R113 1.04 mm to (181.0, 85.3), turned to 90 degrees
- moved C5 0.35 mm to (172.5, 84.3)
- moved C12 0.15 mm to (177.2, 87.3)
- moved U10 0.10 mm to (129.3, 89.4)
Routing:
- net +3V3: track 269.8 -> 271.9 mm, vias 17 -> 18
- net GND: track 248.6 -> 248.3 mm, vias 236 -> 237
